File: RP2350-Daughterboard/RP2350-Daughterboard.kicad_sch (KiCad schematic)
At the start: 77 parts, among them J1 ISA16_DAUGHTER_BUS, J2 SWD, J3 USB-A PORT 1, J4 USB-A PORT 2, J5 HDMI_A, J6 USB 2.0 FRONT PANEL (KEYED), J7 SD_Card_Receptacle, J9 RJ45, SW1 BOOTSEL, SW2 RESET, U1 RP2354B, U10 TPS2051CDBV, U11 ESP32-C3-WROOM-02U, U12 W5500, U2 APS6404L-3SQR-SN, U3 TPD4E05U06DQA, U4 TPD4E05U06DQA, U5 SN74LVC2G07, U6 FE1.1s, U7 TPS2051CDBV, U8 TPS2051CDBV, U9 TPS2051CDBV, Y1 12MHz ABM8-272-T3, Y2 12MHz

Commit message: Added W5500 power
Parts:
- added C34, C36, C37, C38, C39, C40, C41, C46: 100nF, Capacitor_SMD:C_0603_1608Metric, symbol Device:C
- added C35: 10uF, Capacitor_SMD:C_0805_2012Metric, symbol Device:C
- added C42, C48: 4.7uF, Capacitor_SMD:C_0805_2012Metric, symbol Device:C
- added C43, C44: 6.8nF, Capacitor_SMD:C_0603_1608Metric, symbol Device:C
- added C45, C47: 10nF, Capacitor_SMD:C_0603_1608Metric, symbol Device:C
- added L2: 120R @100MHz, Inductor_SMD:L_0603_1608Metric, symbol Device:FerriteBead
- added R20: 12.4k 1%, Resistor_SMD:R_0603_1608Metric, symbol Device:R
- added R21, R22, R24, R25: 49.9R 1%, Resistor_SMD:R_0603_1608Metric, symbol Device:R
- added R23: 10R, Resistor_SMD:R_0603_1608Metric, symbol Device:R
- J9: footprint Connector_RJ:RJ45_Amphenol_54602-x08_Horizontal -> Connector_RJ:RJ45_Amphenol_RJMG1BD3B8K1ANR; symbol Connector:RJ45 -> Connector:RJ45_Amphenol_RJMG1BD3B8K1ANR
Connections:
- net +3V3: now also U12.28 (VDD), U12.43 (PMODE2), U12.44 (PMODE1), U12.45 (PMODE0), C34.1, C35.1, L2.1
- net GND: now also J9.R8, U12.14 (AGND), U12.16 (AGND), U12.19 (AGND), U12.23 (RSVD), U12.29 (GND), U12.3 (AGND), U12.48 (AGND), U12.9 (AGND), C34.2, C35.2, C36.2, C37.2, C38.2, C39.2, C40.2, C41.2, C42.2, C45.2, C46.2, C47.2, C48.2, R20.2
- net ETH_TD_N: now reaches U12.1 (TXN)
- net ETH_TD_N: now also J9.R2 (TD-), R21.2
- net W5500_EXRES: now reaches U12.10 (EXRES1)
- net W5500_EXRES: now also R20.1
- net ETH_3V3A: now reaches U12.11 (AVDD), U12.15 (AVDD), U12.17 (AVDD), U12.21 (AVDD), U12.4 (AVDD), U12.8 (AVDD)
- net ETH_3V3A: now also C36.1, C37.1, C38.1, C39.1, C40.1, C41.1, C48.1, L2.2, R21.1, R22.1, R23.1
- net ETH_TD_P: now reaches U12.2 (TXP)
- net ETH_TD_P: now also J9.R1 (TD+), R22.2
- net W5500_TOCAP: now reaches U12.20 (TOCAP)
- net W5500_TOCAP: now also C42.1
- net W5500_1V2O: now reaches U12.22 (1V2O)
- net W5500_1V2O: now also C47.1
- net ETH_CS_N: now reaches U12.32 (~{SCS})
- net ETH_CS_N: now also U11.6 (IO7)
- net ETH_SCLK: now reaches U12.33 (SCLK)
- net ETH_SCLK: now also U11.3 (IO4)
- net ETH_MISO: now reaches U12.34 (MISO)
- net ETH_MISO: now also U11.5 (IO6)
- net ETH_MOSI: now reaches U12.35 (MOSI)
- net ETH_MOSI: now also U11.4 (IO5)
- net ETH_INT_N: now reaches U12.36 (~{INT})
- net ETH_INT_N: now also U11.15 (IO3)
- net ETH_RST_N: now reaches U12.37 (~{RST})
- net ETH_RST_N: now also U11.10 (IO10)
- net ETH_RXN_SRC: now reaches U12.5 (RXN)
- net ETH_RXN_SRC: now also C44.1, R25.1
- net ETH_RXP_SRC: now reaches U12.6 (RXP)
- net ETH_RXP_SRC: now also C43.1, R24.1
- new net CHASSIS: J9.SH
- new net ETH_CT: C46.1, J9.R4 (TCT), J9.R5 (RCT), R23.2
- new net ETH_RD_N_JACK: C44.2, J9.R6 (RD-)
- new net ETH_RD_P_JACK: C43.2, J9.R3 (RD+)
- new net ETH_RX_BIAS: C45.1, R24.2, R25.2
- no-connect marks 37 -> 48
