File: RP2350-Daughterboard/RP2350-Daughterboard.kicad_sch (KiCad schematic)
At the start: 99 parts, among them J1 ISA16_DAUGHTER_BUS, J2 SWD, J3 USB-A PORT 1, J4 USB-A PORT 2, J5 HDMI_A, J6 USB 2.0 FRONT PANEL (KEYED), J7 SD_Card_Receptacle, J9 RJ45, SW1 BOOTSEL, SW2 RESET, U1 RP2354B, U10 TPS2051CDBV, U11 ESP32-C3-WROOM-02U, U12 W5500, U2 APS6404L-3SQR-SN, U3 TPD4E05U06DQA, U4 TPD4E05U06DQA, U5 SN74LVC2G07, U6 FE1.1s, U7 TPS2051CDBV, U8 TPS2051CDBV, U9 TPS2051CDBV, Y1 12MHz ABM8-272-T3, Y2 12MHz

Commit message: Cleaned up all schematics
Parts:
- removed unit 2 of U5
- removed unit 1 of U5
- added unit 1 of U5
- J1: footprint (none) -> Connector_PCBEdge:BUS_AT
Connections:
- net IRQ_N: now also U5.4 (2Y)
- net RDY: now also U5.6 (1Y)
- net RP_IRQ_DRV: now also U5.3 (2A)
- net RP_RDY_DRV: now also U5.1 (1A)
Other:
- moved on the sheet: C19, C20, C23, C24, C25, C26, C37, C38, C43, C44, C45, C46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
