File: Mainboard/W65C816-Computer.kicad_pcb (KiCad board)
At the start: 2 copper layers, 170 x 170 mm, 107 parts, among them J1 ADDR_DATA_DBG, J2 CTRL_BANK_DBG, J3 CPU_MISC_DBG, J4 PJ-102A, J5 DAUGHTER_PWR_AUX, J6 ISA16_DAUGHTER_BUS, Q1 P-MOSFET_REV_PROT_TO220, SW1 RESET, SW2 NMI, SW3 MAIN_PWR_SW_EXT, U1 W65C816S6PG-14, U10 SN74HC04N, U11 SN74HC08N, U12 SN74HC139N, U2 SN74HC573N, U20 AS6C4008-55PCN, U21 AS6C4008-55PCN, U22 AS6C4008-55PCN, U23 AS6C4008-55PCN, U24 AS6C4008-55PCN, U25 AS6C4008-55PCN, U26 AS6C4008-55PCN, U27 AS6C4008-55PCN, U3 SN74HC245N, U30 SST39VF040-70-4I-NHE, U4 MCP130-315D, U5 SN74HC14N, U6 SN74HC138N, U7 SN74HC138N, U8 SN74HC138N, U9 SN74HC00N, X1 ECS-P143X-8.000-BN

Commit message: Added Readme introduction
Parts:
- removed LED1: PWR, LED_THT:LED_D5.0mm
- removed SW1: RESET, Button_Switch_THT:SW_PUSH_6mm_H4.3mm
- added J7: PWR_LED_HEADER, Connector_PinHeader_2.54mm:PinHeader_1x02_P2.54mm_Vertical, F.Cu at (185.5, 172.7)
- added J8: RESET_HEADER, Connector_PinHeader_2.54mm:PinHeader_1x02_P2.54mm_Vertical, F.Cu at (185.5, 159.6)
- added TP31: U16_OE_N, TestPoint:TestPoint_THTPad_D1.5mm_Drill0.7mm, F.Cu at (161.1, -73.8)
- added TP32: SYS_D0, TestPoint:TestPoint_THTPad_D1.5mm_Drill0.7mm, F.Cu at (161.1, -70.2)
- added TP33: RP_D0, TestPoint:TestPoint_THTPad_D1.5mm_Drill0.7mm, F.Cu at (161.1, -66.7)
- added U16: SN74HC245N, Package_DIP:DIP-20_W7.62mm_Socket_LongPads, F.Cu at (120.1, -80.5)
- added U17: SN74HC32N, Package_DIP:DIP-14_W7.62mm_Socket_LongPads, F.Cu at (134.4, -122.0)
- added U18: SN74HC04N, Package_DIP:DIP-14_W7.62mm_Socket_LongPads, F.Cu at (146.1, -122.0)
- J4: value PJ-102A -> POWER_IN_HEADER_8A; footprint PJ-102A:CUI_PJ-102A -> Connector_Phoenix_MC_HighVoltage:PhoenixContact_MCV_1,5_2-GF-5.08_1x02_P5.08mm_Vertical_ThreadedFlange_MountHole
- moved J4 356.6 mm to (32.9, 163.5), turned to -90 degrees
- moved SW3 336.7 mm to (32.6, 143.7), turned to -90 degrees
- moved F1 313.0 mm to (42.7, 163.6), turned to 90 degrees
- moved J1 272.2 mm to (57.9, -102.3)
- moved J2 258.1 mm to (76.6, -102.3)
- moved D1 252.8 mm to (96.7, -36.8)
- moved U2 244.7 mm to (96.7, -80.5)
- moved U3 244.7 mm to (108.4, -80.5)
- moved C40 218.1 mm to (144.0, -99.9)
- moved C42 218.1 mm to (144.0, -90.3)
- moved C6 211.3 mm to (162.5, -102.6)
- moved R1 207.2 mm to (131.4, -80.6)
- moved R2 207.2 mm to (131.4, -76.6)
- moved R3 207.2 mm to (131.4, -72.5)
- moved R30 207.2 mm to (131.4, -56.3)
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Connections:
- J6 pad 10: /SYS_D3 -> /RP_D3
- J6 pad 12: /SYS_D4 -> /RP_D4
- J6 pad 14: /SYS_D5 -> /RP_D5
- J6 pad 16: /SYS_D6 -> /RP_D6
- J6 pad 18: /SYS_D7 -> /RP_D7
- J6 pad 4: /SYS_D0 -> /RP_D0
- J6 pad 6: /SYS_D1 -> /RP_D1
- J6 pad 8: /SYS_D2 -> /RP_D2
- U12 pad 12: /RP_CS_N -> unconnected-(U12B-O0-Pad12)
Other:
- board text removed: "@Sulfuroid"
- board text removed: "MINI-ITX Kicad Template"

Commit message: Added adapter Gerbers
Parts:
- removed C1, C10, C11, C12, C2, C20, C21, C22, C23, C24, C25, C26, C27, C3, C30, C4, C41, C43, C5, C60, C61, C62, C7, C8, C9: 100nF, Capacitor_THT:C_Disc_D3.0mm_W1.6mm_P2.50mm
- removed C40, C42: 470uF, Capacitor_THT:CP_Radial_D8.0mm_P5.00mm
- removed C6: 10uF, Capacitor_THT:C_Disc_D5.0mm_W2.5mm_P2.50mm
- removed D1: P6KE5.0A, Diode_THT:D_DO-15_P10.16mm_Horizontal
- removed F1: 5A, Fuse:Fuseholder_Clip-5x20mm_Littelfuse_111_Inline_P20.00x5.00mm_D1.05mm_Horizontal
- removed J1: ADDR_DATA_DBG, Connector_PinHeader_2.54mm:PinHeader_1x20_P2.54mm_Vertical
- removed J2: CTRL_BANK_DBG, Connector_PinHeader_2.54mm:PinHeader_1x20_P2.54mm_Vertical
- removed J3: CPU_MISC_DBG, Connector_PinHeader_2.54mm:PinHeader_1x10_P2.54mm_Vertical
- removed J4: POWER_IN_HEADER_8A, Connector_Phoenix_MC_HighVoltage:PhoenixContact_MCV_1,5_2-GF-5.08_1x02_P5.08mm_Vertical_ThreadedFlange_MountHole
- removed J5: DAUGHTER_PWR_AUX, Connector_PinSocket_2.54mm:PinSocket_1x06_P2.54mm_Vertical
- removed J7: PWR_LED_HEADER, Connector_PinHeader_2.54mm:PinHeader_1x02_P2.54mm_Vertical
- removed J8: RESET_HEADER, Connector_PinHeader_2.54mm:PinHeader_1x02_P2.54mm_Vertical
- removed JP1: FLASH_WE_EN, Connector_PinHeader_2.54mm:PinHeader_1x02_P2.54mm_Vertical
- removed MOD1: 3V3_BUCK_MODULE_5V_IN_3A, Connector_PinSocket_2.54mm:PinSocket_1x04_P2.54mm_Vertical
- removed Q1: P-MOSFET_REV_PROT_TO220, Package_TO_SOT_THT:TO-220-3_Vertical
- removed R1, R2, R3, R30, R4, R5, R6: 10k, Resistor_THT:R_Axial_DIN0207_L6.3mm_D2.5mm_P7.62mm_Horizontal
- removed R41: 1k, Resistor_THT:R_Axial_DIN0207_L6.3mm_D2.5mm_P7.62mm_Horizontal
- removed SW2: NMI, Button_Switch_THT:SW_PUSH_6mm_H4.3mm
- removed SW3: MAIN_PWR_SW_EXT, TerminalBlock_RND:TerminalBlock_RND_205-00232_1x02_P5.08mm_Horizontal
- removed TP1: PHI2, TestPoint:TestPoint_THTPad_D1.5mm_Drill0.7mm
- removed TP10: ABORT_N, TestPoint:TestPoint_THTPad_D1.5mm_Drill0.7mm
- removed TP11: PHI2_N, TestPoint:TestPoint_THTPad_D1.5mm_Drill0.7mm
- removed TP12: RAM_CS0_N, TestPoint:TestPoint_THTPad_D1.5mm_Drill0.7mm
- removed TP13: RAM_CS1_N, TestPoint:TestPoint_THTPad_D1.5mm_Drill0.7mm
- removed TP14: RAM_CS2_N, TestPoint:TestPoint_THTPad_D1.5mm_Drill0.7mm
- removed TP15: RAM_CS3_N, TestPoint:TestPoint_THTPad_D1.5mm_Drill0.7mm
- removed TP16: RAM_CS4_N, TestPoint:TestPoint_THTPad_D1.5mm_Drill0.7mm
- removed TP17: RAM_CS5_N, TestPoint:TestPoint_THTPad_D1.5mm_Drill0.7mm
- removed TP18: RAM_CS6_N, TestPoint:TestPoint_THTPad_D1.5mm_Drill0.7mm
- removed TP19: RAM_CS7_N, TestPoint:TestPoint_THTPad_D1.5mm_Drill0.7mm
- removed TP2: RESET_N, TestPoint:TestPoint_THTPad_D1.5mm_Drill0.7mm
- removed TP20: ROM_CS_N, TestPoint:TestPoint_THTPad_D1.5mm_Drill0.7mm
- removed TP21: MEM_OE_N, TestPoint:TestPoint_THTPad_D1.5mm_Drill0.7mm
- removed TP22: MEM_WE_N, TestPoint:TestPoint_THTPad_D1.5mm_Drill0.7mm
- removed TP23: +5V, TestPoint:TestPoint_THTPad_D1.5mm_Drill0.7mm
- removed TP24: +3V3, TestPoint:TestPoint_THTPad_D1.5mm_Drill0.7mm
- removed TP25: GND, TestPoint:TestPoint_THTPad_D1.5mm_Drill0.7mm
- removed TP26: RP_CS_N, TestPoint:TestPoint_THTPad_D1.5mm_Drill0.7mm
- removed TP27: IO_CS_N, TestPoint:TestPoint_THTPad_D1.5mm_Drill0.7mm
- removed TP28: EXP_CS_N, TestPoint:TestPoint_THTPad_D1.5mm_Drill0.7mm
- removed TP29: IO_RD_N, TestPoint:TestPoint_THTPad_D1.5mm_Drill0.7mm
- removed TP3: IRQ_N, TestPoint:TestPoint_THTPad_D1.5mm_Drill0.7mm
- removed TP30: IO_WR_N, TestPoint:TestPoint_THTPad_D1.5mm_Drill0.7mm
- removed TP31: U16_OE_N, TestPoint:TestPoint_THTPad_D1.5mm_Drill0.7mm
- removed TP32: SYS_D0, TestPoint:TestPoint_THTPad_D1.5mm_Drill0.7mm
- removed TP33: RP_D0, TestPoint:TestPoint_THTPad_D1.5mm_Drill0.7mm
- removed TP4: NMI_N, TestPoint:TestPoint_THTPad_D1.5mm_Drill0.7mm
- removed TP5: RDY, TestPoint:TestPoint_THTPad_D1.5mm_Drill0.7mm
- removed TP6: RWB, TestPoint:TestPoint_THTPad_D1.5mm_Drill0.7mm
- removed TP7: VDA, TestPoint:TestPoint_THTPad_D1.5mm_Drill0.7mm
- removed TP8: VPA, TestPoint:TestPoint_THTPad_D1.5mm_Drill0.7mm
- removed TP9: BE, TestPoint:TestPoint_THTPad_D1.5mm_Drill0.7mm
- removed U1: W65C816S6PG-14, Package_DIP:DIP-40_W15.24mm_Socket_LongPads
- removed U10, U18: SN74HC04N, Package_DIP:DIP-14_W7.62mm_Socket_LongPads
- removed U11: SN74HC08N, Package_DIP:DIP-14_W7.62mm_Socket_LongPads
- removed U12: SN74HC139N, Package_DIP:DIP-16_W7.62mm_Socket_LongPads
- removed U16, U3: SN74HC245N, Package_DIP:DIP-20_W7.62mm_Socket_LongPads
- removed U17: SN74HC32N, Package_DIP:DIP-14_W7.62mm_Socket_LongPads
- removed U2: SN74HC573N, Package_DIP:DIP-20_W7.62mm_Socket_LongPads
- removed U20, U21, U22, U23, U24, U25, U26, U27: AS6C4008-55PCN, Package_DIP:DIP-32_W15.24mm_Socket_LongPads
- removed U30: SST39VF040-70-4I-NHE, Package_LCC:PLCC-32_THT-Socket
- removed U4: MCP130-315D, Package_TO_SOT_THT:TO-92_Inline
- removed U5: SN74HC14N, Package_DIP:DIP-14_W7.62mm_Socket_LongPads
- removed U6, U7, U8: SN74HC138N, Package_DIP:DIP-16_W7.62mm_Socket_LongPads
- removed U9: SN74HC00N, Package_DIP:DIP-14_W7.62mm_Socket_LongPads
- removed X1: ECS-P143X-8.000-BN, Oscillator:Oscillator_DIP-14
- moved J6 2.12 mm to (110.6, 183.6)
