File: Mainboard/W65C816-Computer.kicad_sch (KiCad schematic)
At the start: 113 parts, among them J1 ADDR_DATA_DBG, J2 CTRL_BANK_DBG, J3 CPU_MISC_DBG, J4 POWER_IN_HEADER_8A, J5 DAUGHTER_PWR_AUX, J6 ISA16_DAUGHTER_BUS, J7 PWR_LED_HEADER, J8 RESET_HEADER, Q1 P-MOSFET_REV_PROT_TO220, SW2 NMI, SW3 MAIN_PWR_SW_EXT, U1 W65C816S6PG-14, U10 SN74HC04N, U11 SN74HC08N, U12 SN74HC139N, U16 SN74HC245N, U17 SN74HC32N, U18 SN74HC04N, U2 SN74HC573N, U20 AS6C4008-55PCN, U21 AS6C4008-55PCN, U22 AS6C4008-55PCN, U23 AS6C4008-55PCN, U24 AS6C4008-55PCN, U25 AS6C4008-55PCN, U26 AS6C4008-55PCN, U27 AS6C4008-55PCN, U3 SN74HC245N, U30 SST39VF040-70-4I-NHE, U4 MCP130-315D, U5 SN74HC14N, U6 SN74HC138N, U7 SN74HC138N, U8 SN74HC138N, U9 SN74HC00N, X1 ECS-P143X-8.000-BN

Commit message: Cleaned up all schematics
Parts:
- removed C10, C11, C12, C13, C14, C15, C20, C21, C22, C23, C24, C25, C26, C27, C30, C4, C41, C43, C5, C60, C61, C62, C7, C8, C9: 100nF, Capacitor_THT:C_Disc_D3.0mm_W1.6mm_P2.50mm, symbol Device:C
- removed C40, C42: 470uF, Capacitor_THT:CP_Radial_D8.0mm_P5.00mm, symbol Device:C_Polarized
- removed C6: 10uF, Capacitor_THT:C_Disc_D5.0mm_W2.5mm_P2.50mm, symbol Device:C
- removed D1: P6KE5.0A, Diode_THT:D_DO-15_P10.16mm_Horizontal, symbol Device:D_TVS
- removed F1: 5A, Fuse:Fuseholder_Clip-5x20mm_Littelfuse_111_Inline_P20.00x5.00mm_D1.05mm_Horizontal, symbol Device:Fuse
- removed J1: ADDR_DATA_DBG, Connector_PinHeader_2.54mm:PinHeader_1x20_P2.54mm_Vertical, symbol Connector_Generic:Conn_01x20
- removed J2: CTRL_BANK_DBG, Connector_PinHeader_2.54mm:PinHeader_1x20_P2.54mm_Vertical, symbol Connector_Generic:Conn_01x20
- removed J3: CPU_MISC_DBG, Connector_PinHeader_2.54mm:PinHeader_1x10_P2.54mm_Vertical, symbol Connector_Generic:Conn_01x10
- removed J4: POWER_IN_HEADER_8A, Connector_Phoenix_MC_HighVoltage:PhoenixContact_MCV_1,5_2-GF-5.08_1x02_P5.08mm_Vertical_ThreadedFlange_MountHole, symbol Connector_Generic:Conn_01x02
- removed J5: DAUGHTER_PWR_AUX, Connector_PinSocket_2.54mm:PinSocket_1x06_P2.54mm_Vertical, symbol Connector_Generic:Conn_01x06
- removed J7: PWR_LED_HEADER, Connector_PinHeader_2.54mm:PinHeader_1x02_P2.54mm_Vertical, symbol Connector_Generic:Conn_01x02
- removed J8: RESET_HEADER, Connector_PinHeader_2.54mm:PinHeader_1x02_P2.54mm_Vertical, symbol Connector_Generic:Conn_01x02
- removed JP1: FLASH_WE_EN, Connector_PinHeader_2.54mm:PinHeader_1x02_P2.54mm_Vertical, symbol Connector_Generic:Conn_01x02
- removed MOD1: 3V3_BUCK_MODULE_5V_IN_3A, Connector_PinSocket_2.54mm:PinSocket_1x04_P2.54mm_Vertical, symbol Connector_Generic:Conn_01x04
- removed Q1: P-MOSFET_REV_PROT_TO220, Package_TO_SOT_THT:TO-220-3_Vertical, symbol Transistor_FET:Q_PMOS_GDS
- removed R2, R3, R30, R4, R5, R6, R7: 10k, Resistor_THT:R_Axial_DIN0207_L6.3mm_D2.5mm_P7.62mm_Horizontal, symbol Device:R
- removed R41: 1k, Resistor_THT:R_Axial_DIN0207_L6.3mm_D2.5mm_P7.62mm_Horizontal, symbol Device:R
- removed SW2: NMI, Button_Switch_THT:SW_PUSH_6mm_H4.3mm, symbol Switch:SW_Push
- removed SW3: MAIN_PWR_SW_EXT, TerminalBlock_RND:TerminalBlock_RND_205-00232_1x02_P5.08mm_Horizontal, symbol Switch:SW_SPST
- removed TP1: PHI2, TestPoint:TestPoint_THTPad_D1.5mm_Drill0.7mm, symbol Connector:TestPoint
- removed TP10: ABORT_N, TestPoint:TestPoint_THTPad_D1.5mm_Drill0.7mm, symbol Connector:TestPoint
- removed TP11: PHI2_N, TestPoint:TestPoint_THTPad_D1.5mm_Drill0.7mm, symbol Connector:TestPoint
- removed TP12: RAM_CS0_N, TestPoint:TestPoint_THTPad_D1.5mm_Drill0.7mm, symbol Connector:TestPoint
- removed TP13: RAM_CS1_N, TestPoint:TestPoint_THTPad_D1.5mm_Drill0.7mm, symbol Connector:TestPoint
- removed TP14: RAM_CS2_N, TestPoint:TestPoint_THTPad_D1.5mm_Drill0.7mm, symbol Connector:TestPoint
- removed TP15: RAM_CS3_N, TestPoint:TestPoint_THTPad_D1.5mm_Drill0.7mm, symbol Connector:TestPoint
- removed TP16: RAM_CS4_N, TestPoint:TestPoint_THTPad_D1.5mm_Drill0.7mm, symbol Connector:TestPoint
- removed TP17: RAM_CS5_N, TestPoint:TestPoint_THTPad_D1.5mm_Drill0.7mm, symbol Connector:TestPoint
- removed TP18: RAM_CS6_N, TestPoint:TestPoint_THTPad_D1.5mm_Drill0.7mm, symbol Connector:TestPoint
- removed TP19: RAM_CS7_N, TestPoint:TestPoint_THTPad_D1.5mm_Drill0.7mm, symbol Connector:TestPoint
- removed TP2: RESET_N, TestPoint:TestPoint_THTPad_D1.5mm_Drill0.7mm, symbol Connector:TestPoint
- removed TP20: ROM_CS_N, TestPoint:TestPoint_THTPad_D1.5mm_Drill0.7mm, symbol Connector:TestPoint
- removed TP21: MEM_OE_N, TestPoint:TestPoint_THTPad_D1.5mm_Drill0.7mm, symbol Connector:TestPoint
- removed TP22: MEM_WE_N, TestPoint:TestPoint_THTPad_D1.5mm_Drill0.7mm, symbol Connector:TestPoint
- removed TP23: +5V, TestPoint:TestPoint_THTPad_D1.5mm_Drill0.7mm, symbol Connector:TestPoint
- removed TP24: +3V3, TestPoint:TestPoint_THTPad_D1.5mm_Drill0.7mm, symbol Connector:TestPoint
- removed TP25: GND, TestPoint:TestPoint_THTPad_D1.5mm_Drill0.7mm, symbol Connector:TestPoint
- removed TP26: RP_CS_N, TestPoint:TestPoint_THTPad_D1.5mm_Drill0.7mm, symbol Connector:TestPoint
- removed TP27: IO_CS_N, TestPoint:TestPoint_THTPad_D1.5mm_Drill0.7mm, symbol Connector:TestPoint
- removed TP28: EXP_CS_N, TestPoint:TestPoint_THTPad_D1.5mm_Drill0.7mm, symbol Connector:TestPoint
- removed TP29: IO_RD_N, TestPoint:TestPoint_THTPad_D1.5mm_Drill0.7mm, symbol Connector:TestPoint
- removed TP3: IRQ_N, TestPoint:TestPoint_THTPad_D1.5mm_Drill0.7mm, symbol Connector:TestPoint
- removed TP30: IO_WR_N, TestPoint:TestPoint_THTPad_D1.5mm_Drill0.7mm, symbol Connector:TestPoint
- removed TP31: U16_OE_N, TestPoint:TestPoint_THTPad_D1.5mm_Drill0.7mm, symbol Connector:TestPoint
- removed TP32: SYS_D0, TestPoint:TestPoint_THTPad_D1.5mm_Drill0.7mm, symbol Connector:TestPoint
- removed TP33: RP_D0, TestPoint:TestPoint_THTPad_D1.5mm_Drill0.7mm, symbol Connector:TestPoint
- removed TP4: NMI_N, TestPoint:TestPoint_THTPad_D1.5mm_Drill0.7mm, symbol Connector:TestPoint
- removed TP5: RDY, TestPoint:TestPoint_THTPad_D1.5mm_Drill0.7mm, symbol Connector:TestPoint
- removed TP6: RWB, TestPoint:TestPoint_THTPad_D1.5mm_Drill0.7mm, symbol Connector:TestPoint
- removed TP7: VDA, TestPoint:TestPoint_THTPad_D1.5mm_Drill0.7mm, symbol Connector:TestPoint
- removed TP8: VPA, TestPoint:TestPoint_THTPad_D1.5mm_Drill0.7mm, symbol Connector:TestPoint
- removed TP9: BE, TestPoint:TestPoint_THTPad_D1.5mm_Drill0.7mm, symbol Connector:TestPoint
- removed U10, U18: SN74HC04N, Package_DIP:DIP-14_W7.62mm_Socket_LongPads, symbol 74xx:74HC04
- removed U11: SN74HC08N, Package_DIP:DIP-14_W7.62mm_Socket_LongPads, symbol W65C816-Computer:74HC08
- removed U12: SN74HC139N, Package_DIP:DIP-16_W7.62mm_Socket_LongPads, symbol 74xx:74LS139
- removed U16: SN74HC245N, Package_DIP:DIP-20_W7.62mm_Socket_LongPads, symbol 74xx:74HC245
- removed U17: SN74HC32N, Package_DIP:DIP-14_W7.62mm_Socket_LongPads, symbol W65C816-Computer:74HC32
- removed U30: SST39VF040-70-4I-NHE, Package_LCC:PLCC-32_THT-Socket, symbol Memory_Flash:SST39SF040
- removed U4: MCP130-315D, Package_TO_SOT_THT:TO-92_Inline, symbol Power_Supervisor:MCP130-xxxDxTO
- removed U5: SN74HC14N, Package_DIP:DIP-14_W7.62mm_Socket_LongPads, symbol 74xx:74HC14
- removed U6, U7, U8: SN74HC138N, Package_DIP:DIP-16_W7.62mm_Socket_LongPads, symbol 74xx:74HC138
- removed U9: SN74HC00N, Package_DIP:DIP-14_W7.62mm_Socket_LongPads, symbol 74xx:74HC00
- removed X1: ECS-P143X-8.000-BN, Oscillator:Oscillator_DIP-14, symbol Oscillator:CXO_DIP14
- added U18: SN74AHC04N, SN74AHC04N:DIP794W45P254L1969H508Q14, symbol SN74AHC04N:SN74AHC04N
- C1, C2, C3: footprint Capacitor_THT:C_Disc_D3.0mm_W1.6mm_P2.50mm -> (none)
- R1: footprint Resistor_THT:R_Axial_DIN0207_L6.3mm_D2.5mm_P7.62mm_Horizontal -> (none)
- U1: symbol W65C816-Computer:W65C816S6PG-14 -> W65C816-Computer:W65C816S6PG_14_Readable_v2
- U2: value SN74HC573N -> 74LS573; footprint Package_DIP:DIP-20_W7.62mm_Socket_LongPads -> (none)
- U3: value SN74HC245N -> 74HC245; footprint Package_DIP:DIP-20_W7.62mm_Socket_LongPads -> (none)
Connections:
- net RAM_CS1_N is gone; now on net RAM_CS0_N: U21.22 (CE#)
- net RAM_CS2_N is gone; now on net RAM_CS0_N: U22.22 (CE#)
- net RAM_CS3_N is gone; now on net RAM_CS0_N: U23.22 (CE#)
- net RAM_CS4_N is gone; now on net RAM_CS0_N: U24.22 (CE#)
- net RAM_CS5_N is gone; now on net RAM_CS0_N: U25.22 (CE#)
- net RAM_CS6_N is gone; now on net RAM_CS0_N: U26.22 (CE#)
- net RAM_CS7_N is gone; now on net RAM_CS0_N: U27.22 (CE#)
- net +3V3: no longer C1.1, C2.1, C3.1, R1.1, U1.8 (VDD), U2.20 (VCC), U20.32 (VCC), U21.32 (VCC), U22.32 (VCC), U23.32 (VCC), U24.32 (VCC), U25.32 (VCC), U26.32 (VCC), U27.32 (VCC), U3.20 (VCC)
- net +5V: now also C1.1, C2.1, C3.1, R1.1, U1.8 (VDD), U2.20 (VCC), U20.32 (VCC), U21.32 (VCC), U22.32 (VCC), U23.32 (VCC), U24.32 (VCC), U25.32 (VCC), U26.32 (VCC), U27.32 (VCC), U3.20 (VCC), U18.14 (VCC)
- net GND: now also U18.11 (5A), U18.13 (6A), U18.3 (2A), U18.5 (3A), U18.7 (GND), U18.9 (4A)
- net IRQ_N: now also U1.6 (NMI_N); no longer U1.4 (IRQB)
- net NMI_N: now also U1.4 (IRQ_N); no longer U1.6 (NMIB)
- net PHI2: now also U18.1 (1A)
- net PHI2_N: now also U18.2 (1Y); no longer U3.19 (CE)
- net D0 renamed CPU_D0
- net D1 renamed CPU_D1
- net D2 renamed CPU_D2
- net D3 renamed CPU_D3
- net D4 renamed CPU_D4
- net D5 renamed CPU_D5
- net D6 renamed CPU_D6
- net D7 renamed CPU_D7
- net RESET_RC renamed MEM_DATA_OE_N
- net MEM_DATA_OE_N: now also U3.19 (CE)
- no-connect marks 55 -> 23
Other:
- note added: "RAM DEFAULT CLUSTER"
- note added: "RAM EXPANSION CLUSTER"
- note removed: "Power input: PJ-102A barrel jack is center-positive and rated 2.5 A. +5V is fused, switched, reverse-polarity protected by Q1, TVS-clamped, then feeds the daughterboard power connector and MOD1 3.3 V buck module."
- note removed: "Rev A decode: U7 divides low 4 MB into 512 KB SRAM banks; U6 detects bank $00. Flash overlays $00:8000-$FFFF for reset vectors. U9 disables RAM0 while ROM is active. MEM_OE_N=!RWB, MEM_WE_N=RWB."
- note removed: "SRAM sockets U21-U27 complete 4 MB main SRAM bank with U20"
- note removed: "Stage 1 subsystem: W65C816S, 8 MHz 3.3 V clock, MCP130 reset, 74HC573 bank latch, one AS6C4008 SRAM, SST39VF040 boot Flash. RP2350/video not populated here."
- moved on the sheet: U20
